File: pcb/Power-main/ver0.1/Power-main.kicad_pcb (KiCad board)
At the start: 2 copper layers, 2 parts, among them U1 LM5143QRHARQ1, U2 TPS54335ADDAR

Commit message: 提交测试
Parts:
- added U1: LM5143QRHARQ1, BuckConvert:LM5143QRHARQ1, F.Cu at (99.1, 51.1)
- added U1: LM5143QRHARQ1, BuckConvert:LM5143QRHARQ1, F.Cu at (87.1, 67.1)
- added U1: LM5143QRHARQ1, BuckConvert:LM5143QRHARQ1, F.Cu at (70.5, 51.1)

Commit message: 提交测试
Parts:
- removed the U1 at (99.1, 51.1)
- removed the U1 at (87.1, 67.1)
- removed the U1 at (70.5, 51.1)
- added U1: LM5143QRHARQ1, BuckConvert:LM5143QRHARQ1, F.Cu at (69.5, 53.7)
